File: kicad/wireless_adapter_for_mitsubishi/connector_wr.kicad_sch (KiCad schematic)
At the start: 7 parts, among them J2 S05B-PASK-2(LF)(SN), U5 TVS1400DRVR, U6 TVS0500DRVR

Commit message: Rename some KiCad buses.
Connections:
- net WR_RX_WA_TX renamed WR_UART_RX
- net WR_TX_WA_RX renamed WR_UART_TX
Changed lines of the file:
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@@
 		)
 	)
-	(hierarchical_label "WR_RX_WA_TX"
+	(hierarchical_label "WR_UART_RX"
 		(shape input)
 		(at 205.74 86.36 0)
@@
 		)
 	)
-	(hierarchical_label "WR_TX_WA_RX"
-		(shape input)
+	(hierarchical_label "WR_UART_TX"
+		(shape output)
 		(at 205.74 99.06 0)
 		(effects
