File: kicad/wireless_adapter_for_mitsubishi/power_subsystem.kicad_sch (KiCad schematic)
At the start: 16 parts, among them U7 TPS2121RUXR, U8 TPSM5601R5HRDAR

Commit message: Clean up KiCad schematic.
Connections:
- net Power_Multiplexed renamed Multiplexer_Output
Other:
- note added: "3.3V Output Switching Voltage Regulator"
- note added: "CISPR 22 CLASS B EMI Filter"
- note added: "IU/USB Power Multiplexer"
- note removed: "3.3V Output Switching Voltage Regulator."
- note removed: "CISPR 22 CLASS B EMI Filter for the Switching Voltage Regulator."
- note removed: "IU/USB Power Multiplexer."
- moved on the sheet: C10, C11, C12, C13, C14, C15, C7, C8, C9, L1, R10, R11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
