File: kicad/wireless_adapter_for_mitsubishi/wireless_adapter_for_mitsubishi.kicad_sch (KiCad schematic)
At the start: 17 parts, among them U1 ESP32-C6-WROOM-1-N8, U2 TXS0104EPWR

Commit message: Rename some of the KiCad sheets.
Other:
- sheet Power Regulator renamed Power System
- sheet Power System: file power_regulator.kicad_sch -> power_subsystem.kicad_sch
- sheet WR Connector: file connector_mhk.kicad_sch -> connector_wr.kicad_sch
Changed lines of the file:
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@@
 		)
 		(instances
-			(project "mitsubishi_wireless_adapter"
+			(project "wireless_adapter_for_mitsubishi"
 				(path "/f70a83b0-34a1-41b3-a332-066c3f3f3918"
 					(reference "#PWR01")
@@
 		)
 		(instances
-			(project "mitsubishi_wireless_adapter"
+			(project "wireless_adapter_for_mitsubishi"
 				(path "/f70a83b0-34a1-41b3-a332-066c3f3f3918"
 					(reference "#PWR021")
@@
 		)
 		(instances
-			(project "mitsubishi_wireless_adapter"
+			(project "wireless_adapter_for_mitsubishi"
 				(path "/f70a83b0-34a1-41b3-a332-066c3f3f3918"
 					(reference "C2")
@@
 		)
 		(instances
-			(project "mitsubishi_wireless_adapter"
+			(project "wireless_adapter_for_mitsubishi"
 				(path "/f70a83b0-34a1-41b3-a332-066c3f3f3918"
 					(reference "#PWR034")
@@
 		)
 		(instances
-			(project "mitsubishi_wireless_adapter"
+			(project "wireless_adapter_for_mitsubishi"
 				(path "/f70a83b0-34a1-41b3-a332-066c3f3f3918"
 					(reference "R2")
@@
 		)
 		(instances
-			(project "mitsubishi_wireless_adapter"
+			(project "wireless_adapter_for_mitsubishi"
 				(path "/f70a83b0-34a1-41b3-a332-066c3f3f3918"
 					(reference "#PWR020")
@@
 		)
 		(instances
-			(project "mitsubishi_wireless_adapter"
+			(project "wireless_adapter_for_mitsubishi"
 				(path "/f70a83b0-34a1-41b3-a332-066c3f3f3918"
 					(reference "#PWR045")
@@
 		)
 		(instances
-			(project "mitsubishi_wireless_adapter"
+			(project "wireless_adapter_for_mitsubishi"
 				(path "/f70a83b0-34a1-41b3-a332-066c3f3f3918"
 					(reference "U2")
@@
 		)
 		(instances
-			(project "mitsubishi_wireless_adapter"
+			(project "wireless_adapter_for_mitsubishi"
 				(path "/f70a83b0-34a1-41b3-a332-066c3f3f3918"
 					(reference "#PWR016")
@@
 		)
 		(instances
-			(project "mitsubishi_wireless_adapter"
+			(project "wireless_adapter_for_mitsubishi"
 				(path "/f70a83b0-34a1-41b3-a332-066c3f3f3918"
 					(reference "#PWR09")
@@
 		)
 		(instances
-			(project "mitsubishi_wireless_adapter"
+			(project "wireless_adapter_for_mitsubishi"
 				(path "/f70a83b0-34a1-41b3-a332-066c3f3f3918"
 					(reference "C3")
@@
 		)
 		(instances
-			(project "mitsubishi_wireless_adapter"
+			(project "wireless_adapter_for_mitsubishi"
 				(path "/f70a83b0-34a1-41b3-a332-066c3f3f3918"
 					(reference "#PWR019")
@@
 		)
 		(instances
-			(project "mitsubishi_wireless_adapter"
+			(project "wireless_adapter_for_mitsubishi"
 				(path "/f70a83b0-34a1-41b3-a332-066c3f3f3918"
 					(reference "#PWR022")
@@
 		)
 		(instances
-			(project "mitsubishi_wireless_adapter"
+			(project "wireless_adapter_for_mitsubishi"
 				(path "/f70a83b0-34a1-41b3-a332-066c3f3f3918"
 					(reference "#PWR010")
@@
 		)
 		(instances
-			(project "mitsubishi_wireless_adapter"
+			(project "wireless_adapter_for_mitsubishi"
 				(path "/f70a83b0-34a1-41b3-a332-066c3f3f3918"
 					(reference "R1")
@@
 		)
 		(instances
-			(project "mitsubishi_wireless_adapter"
+			(project "wireless_adapter_for_mitsubishi"
 				(path "/f70a83b0-34a1-41b3-a332-066c3f3f3918"
 					(reference "H2")
@@
 		)
 		(instances
-			(project "mitsubishi_wireless_adapter"
+			(project "wireless_adapter_for_mitsubishi"
 				(path "/f70a83b0-34a1-41b3-a332-066c3f3f3918"
 					(reference "#PWR013")
@@
 		)
 		(instances
-			(project "mitsubishi_wireless_adapter"
+			(project "wireless_adapter_for_mitsubishi"
 				(path "/f70a83b0-34a1-41b3-a332-066c3f3f3918"
 					(reference "#PWR015")
@@
 		)
 		(instances
-			(project "mitsubishi_wireless_adapter"
+			(project "wireless_adapter_for_mitsubishi"
 				(path "/f70a83b0-34a1-41b3-a332-066c3f3f3918"
 					(reference "H3")
@@
 		)
 		(instances
-			(project "mitsubishi_wireless_adapter"
+			(project "wireless_adapter_for_mitsubishi"
 				(path "/f70a83b0-34a1-41b3-a332-066c3f3f3918"
 					(reference "#PWR07")
@@
 		)
 		(instances
-			(project "mitsubishi_wireless_adapter"
+			(project "wireless_adapter_for_mitsubishi"
 				(path "/f70a83b0-34a1-41b3-a332-066c3f3f3918"
 					(reference "#PWR011")
@@
 		)
 		(instances
-			(project "mitsubishi_wireless_adapter"
+			(project "wireless_adapter_for_mitsubishi"
 				(path "/f70a83b0-34a1-41b3-a332-066c3f3f3918"
 					(reference "#PWR018")
@@
 		)
 		(instances
-			(project "mitsubishi_wireless_adapter"
+			(project "wireless_adapter_for_mitsubishi"
 				(path "/f70a83b0-34a1-41b3-a332-066c3f3f3918"
 					(reference "C4")
@@
 		)
 		(instances
-			(project "mitsubishi_wireless_adapter"
+			(project "wireless_adapter_for_mitsubishi"
 				(path "/f70a83b0-34a1-41b3-a332-066c3f3f3918"
 					(reference "S1")
@@
 		)
 		(instances
-			(project "mitsubishi_wireless_adapter"
+			(project "wireless_adapter_for_mitsubishi"
 				(path "/f70a83b0-34a1-41b3-a332-066c3f3f3918"
 					(reference "#PWR038")
@@
 		)
 		(instances
-			(project "mitsubishi_wireless_adapter"
+			(project "wireless_adapter_for_mitsubishi"
 				(path "/f70a83b0-34a1-41b3-a332-066c3f3f3918"
 					(reference "R3")
@@
 		)
 		(instances
-			(project "mitsubishi_wireless_adapter"
+			(project "wireless_adapter_for_mitsubishi"
 				(path "/f70a83b0-34a1-41b3-a332-066c3f3f3918"
 					(reference "C5")
@@
 		)
 		(instances
-			(project "mitsubishi_wireless_adapter"
+			(project "wireless_adapter_for_mitsubishi"
 				(path "/f70a83b0-34a1-41b3-a332-066c3f3f3918"
 					(reference "#PWR03")
@@
 		)
 		(instances
-			(project "mitsubishi_wireless_adapter"
+			(project "wireless_adapter_for_mitsubishi"
 				(path "/f70a83b0-34a1-41b3-a332-066c3f3f3918"
 					(reference "H4")
@@
 		)
 		(instances
-			(project "mitsubishi_wireless_adapter"
+			(project "wireless_adapter_for_mitsubishi"
 				(path "/f70a83b0-34a1-41b3-a332-066c3f3f3918"
 					(reference "S2")
@@
 		)
 		(instances
-			(project "mitsubishi_wireless_adapter"
+			(project "wireless_adapter_for_mitsubishi"
 				(path "/f70a83b0-34a1-41b3-a332-066c3f3f3918"
 					(reference "H1")
@@
 		)
 		(instances
-			(project "mitsubishi_wireless_adapter"
+			(project "wireless_adapter_for_mitsubishi"
 				(path "/f70a83b0-34a1-41b3-a332-066c3f3f3918"
 					(reference "C6")
@@
 		)
 		(instances
-			(project "mitsubishi_wireless_adapter"
+			(project "wireless_adapter_for_mitsubishi"
 				(path "/f70a83b0-34a1-41b3-a332-066c3f3f3918"
 					(reference "#PWR044")
@@
 		)
 		(instances
-			(project "mitsubishi_wireless_adapter"
+			(project "wireless_adapter_for_mitsubishi"
 				(path "/f70a83b0-34a1-41b3-a332-066c3f3f3918"
 					(reference "#PWR039")
@@
 		)
 		(instances
-			(project "mitsubishi_wireless_adapter"
+			(project "wireless_adapter_for_mitsubishi"
 				(path "/f70a83b0-34a1-41b3-a332-066c3f3f3918"
 					(reference "#PWR025")
@@
 		)
 		(instances
-			(project "mitsubishi_wireless_adapter"
+			(project "wireless_adapter_for_mitsubishi"
 				(path "/f70a83b0-34a1-41b3-a332-066c3f3f3918"
 					(reference "#PWR023")
@@
 		)
 		(instances
-			(project "mitsubishi_wireless_adapter"
+			(project "wireless_adapter_for_mitsubishi"
 				(path "/f70a83b0-34a1-41b3-a332-066c3f3f3918"
 					(reference "U1")
@@
 		)
 		(instances
-			(project "mitsubishi_wireless_adapter"
+			(project "wireless_adapter_for_mitsubishi"
 				(path "/f70a83b0-34a1-41b3-a332-066c3f3f3918"
 					(reference "C1")
@@
 		)
 		(instances
-			(project "mitsubishi_wireless_adapter"
+			(project "wireless_adapter_for_mitsubishi"
 				(path "/f70a83b0-34a1-41b3-a332-066c3f3f3918"
 					(page "2")
@@
 			(color 0 0 0 0)
 		)
-		(property "Sheetname" "Power Regulator"
+		(property "Sheetname" "Power System"
 			(at 60.96 42.672 0)
 			(show_name no)
@@
 			)
 		)
-		(property "Sheetfile" "power_regulator.kicad_sch"
+		(property "Sheetfile" "power_subsystem.kicad_sch"
 			(at 66.04 59.182 0)
 			(hide yes)
@@
 		)
 		(instances
-			(project "mitsubishi_wireless_adapter"
+			(project "wireless_adapter_for_mitsubishi"
 				(path "/f70a83b0-34a1-41b3-a332-066c3f3f3918"
 					(page "5")
@@
 			)
 		)
-		(property "Sheetfile" "connector_mhk.kicad_sch"
+		(property "Sheetfile" "connector_wr.kicad_sch"
 			(at 30.48 117.348 0)
 			(hide yes)
@@
 		)
 		(instances
-			(project "mitsubishi_wireless_adapter"
+			(project "wireless_adapter_for_mitsubishi"
 				(path "/f70a83b0-34a1-41b3-a332-066c3f3f3918"
 					(page "3")
@@
 		)
 		(instances
-			(project "mitsubishi_wireless_adapter"
+			(project "wireless_adapter_for_mitsubishi"
 				(path "/f70a83b0-34a1-41b3-a332-066c3f3f3918"
 					(page "4")

Commit message: Fix the name of a KiCad sheet.
Other:
- sheet Power System renamed Power Subsystem
Changed lines of the file:
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@@
 			(color 0 0 0 0)
 		)
-		(property "Sheetname" "Power System"
+		(property "Sheetname" "Power Subsystem"
 			(at 60.96 42.672 0)
 			(show_name no)

Commit message: Rename some KiCad buses.
Connections:
- net IU Connector/IU_RX_WA_TX renamed IU Connector/IU_UART_RX
- net IU Connector/IU_TX_WA_RX renamed IU Connector/IU_UART_TX
- net WR Connector/WR_RX_WA_TX renamed WR Connector/WR_UART_RX
- net WR Connector/WR_TX_WA_RX renamed WR Connector/WR_UART_TX
Other:
- sheet IU Connector ports: added IU_UART_RX, IU_UART_TX; removed IU_RX_WA_TX, IU_TX_WA_RX
- sheet WR Connector ports: added WR_UART_RX, WR_UART_TX; removed WR_RX_WA_TX, WR_TX_WA_RX
Changed lines of the file:
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@@
 			)
 		)
-		(pin "IU_RX_WA_TX" output
+		(pin "IU_UART_RX" input
 			(at 38.1 76.2 0)
 			(effects
@@
 			)
 		)
-		(pin "IU_TX_WA_RX" output
+		(pin "IU_UART_TX" output
 			(at 38.1 73.66 0)
 			(effects
@@
 			)
 		)
-		(pin "WR_RX_WA_TX" input
+		(pin "WR_UART_RX" input
 			(at 38.1 106.68 0)
 			(effects
@@
 			)
 		)
-		(pin "WR_TX_WA_RX" input
+		(pin "WR_UART_TX" output
 			(at 38.1 109.22 0)
 			(effects

Commit message: Clean up KiCad schematic.
Other:
- note added: "Firmware Development, Debug and Recovery"
- note added: "Mounting Holes"
- note added: "Operational Connectors"
- note added: "Power Source Multiplexing and Voltage Step Down"
- note added: "System on a Chip (SoC)"
- moved on the sheet: C1, C2, C5, C6, R1, R2, S1, S2, U2

Commit message: Flatten KiCad schematic.
Parts:
- added C10, C11: 2.2μF, Capacitor_SMD:C_1206_3216Metric, symbol Project:Samsung_CL31B225KBHNNNE
- added C12, C13: 22nF, Capacitor_SMD:C_0603_1608Metric, symbol Project:Samsung_CL10B223KB8NNNC
- added C14, C15: 47μF, Capacitor_SMD:C_1206_3216Metric, symbol Project:Samsung_CL31A476MPHNNNE
- added C7: 1μF, Project:C_0402_1005Metric, symbol Project:Samsung_CL05A105KA5NQNC
- added C8, C9: 10μF, Capacitor_SMD:C_1206_3216Metric, symbol Project:Samsung_CL31A106KBHNNNE
- added D1, D2, D3, D4, D5, D6, D7: H5VL10B, Diode_SMD:D_SOD-882, symbol Project:RNO_H5VL10B
- added J1, J2: S05B-PASK-2(LF)(SN), Project:JST_PA_S05B-PASK-2_1x05_P2.00mm_Horizontal, symbol Project:JST_S05B-PASK-2(LF)(SN)
- added J3: GT-USB-7010ASV, Project:USB_C_Receptacle_G-Switch_GT-USB-7010ASV, symbol Project:G-Switch_GT-USB-7010ASV
- added L1: 470nH, Project:L_0806_2016Metric, symbol Project:Murata_DFE201610E-R47M=P2
- added R10: 100kΩ(1%), Project:R_0402_1005Metric, symbol Project:Uniroyal_0402WGF1003TCE
- added R11: 100mΩ, Resistor_SMD:R_1206_3216Metric, symbol Project:Uniroyal_1206W4F100LT5E
- added R12: 51kΩ(1%), Project:R_0402_1005Metric, symbol Project:Uniroyal_0402WGF5102TCE
- added R13: 22kΩ(1%), Project:R_0402_1005Metric, symbol Project:Uniroyal_0402WGF2202TCE
- added R4, R5, R6, R7: 470Ω, Project:R_0402_1005Metric, symbol Project:Uniroyal_0402WGF4700TCE
- added R8, R9: 5.1kΩ(1%), Project:R_0402_1005Metric, symbol Project:Uniroyal_0402WGF4700TCE
- added U3, U5: TVS1400DRVR, Package_SON:WSON-6-1EP_2x2mm_P0.65mm_EP1x1.6mm, symbol Project:Texas_TVS1400DRVR
- added U4, U6: TVS0500DRVR, Package_SON:WSON-6-1EP_2x2mm_P0.65mm_EP1x1.6mm, symbol Project:Texas_TVS0500DRVR
- added U7: TPS2121RUXR, Project:Texas_RUX0012A_VQFN-HR-12_2x2.5x1mm_P0.5mm, symbol Project:Texas_TPS2121RUXT
- added U8: TPSM5601R5HRDAR, Project:Texas_RDA0015A_B3QFN-14-1EP_5x5.5x4.1mm_P0.65mm, symbol Project:Texas_TPSM5601R5HRDAR
Connections:
- net +3V3: now also C14.1, C15.1, R12.1, U8.7 (VOUT), U8.8 (VOUT)
- net GND: now also C10.2, C11.2, C12.2, C13.2, C14.2, C15.2, C7.2, C8.2, C9.2, D1.2 (A2), D2.2 (A2), D3.2 (A2), D4.2 (A2), D5.2 (A2), D6.2 (A2), D7.2 (A2), J1.2 (Pin_2), J2.2 (Pin_2), J3.A1 (GND), J3.A12 (GND), J3.B1 (GND), J3.B12 (GND), J3.SH (SHIELD), R10.2, R13.2, R8.2, R9.2, U3.1 (GND), U3.2 (GND), U3.3 (GND), U3.7 (GND), U4.1 (GND), U4.2 (GND), U4.3 (GND), U4.7 (GND), U5.1 (GND), U5.2 (GND), U5.3 (GND), U5.7 (GND), U6.1 (GND), U6.2 (GND), U6.3 (GND), U6.7 (GND), U7.12 (GND), U7.3 (CP2), U7.4 (OV2), U7.5 (OV1), U7.6 (PR1), U7.9 (ST), U8.10 (AGND), U8.15 (PGND)
- net USB_D+: now also D7.1 (A1), J3.A6 (D+), J3.B6 (D+)
- net USB_D-: now also D6.1 (A1), J3.A7 (D-), J3.B7 (D-)
- net IU Connector/IU_5V renamed IU_5V
- net IU_5V: now also J1.3 (Pin_3), J2.3 (Pin_3), U4.4 (IN), U4.5 (IN), U4.6 (IN), U6.4 (IN), U6.5 (IN), U6.6 (IN)
- net IU Connector/IU_UART_RX: no longer names the net of U2.3 (A2)
- net IU Connector/IU_UART_RX: now also R5.2
- net IU Connector/IU_UART_TX: no longer names the net of U2.2 (A1)
- net IU Connector/IU_UART_TX: now also R4.2
- net WR Connector/WR_UART_RX: no longer names the net of U2.4 (A3)
- net WR Connector/WR_UART_RX: now also R6.2
- net WR Connector/WR_UART_TX: no longer names the net of U2.5 (A4)
- net WR Connector/WR_UART_TX: now also R7.2
- new net: D2.1 (A1), J1.5 (Pin_5), R5.1
- new net: D3.1 (A1), J2.4 (Pin_4), R6.1
- new net: J3.A5 (CC1), R9.1
- new net: J3.B5 (CC2), R8.1
- new net: D1.1 (A1), J1.4 (Pin_4), R4.1
- new net: C7.1, U7.11 (SS)
- new net: U8.13 (NC), U8.3 (NC), U8.6 (NC)
- new net: R12.2, R13.1, U8.9 (FB)
- new net: D4.1 (A1), J2.5 (Pin_5), R7.1
- new net: C9.1, R11.2
- new net: R10.1, U7.10 (ILIM)
- new net IU_12V7: J1.1 (Pin_1), J2.1 (Pin_1), U3.4 (IN), U3.5 (IN), U3.6 (IN), U5.4 (IN), U5.5 (IN), U5.6 (IN), U7.7 (IN1)
- new net Multiplexer_Output: C8.1, L1.1, U7.1 (OUT), U7.8 (OUT)
- new net Regulator_Input: C10.1, C11.1, C12.1, C13.1, L1.2, R11.1, U8.1 (VIN), U8.14 (VIN), U8.2 (EN)
- new net USB_5V: D5.1 (A1), J3.A4 (VBUS), J3.A9 (VBUS), J3.B4 (VBUS), J3.B9 (VBUS), U7.2 (IN2)
- no-connect marks 15 -> 22
Other:
- removed sheet IU Connector
- removed sheet Power Subsystem
- removed sheet USB Connector
- removed sheet WR Connector
- note added: "3.3V Output Switching Voltage Regulator"
- note added: "CISPR 22 CLASS B EMI Filter"
- note added: "Connect AGND to GND (PGND) at a single point."
- note added: "IU/USB Power Multiplexer"
- note removed: "Power Source Multiplexing and Voltage Step Down"
- moved on the sheet: C1, C2, C3, C4, C5, C6, R1, R2, R3, S1, S2, U1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

Commit message: Clean up KiCad schematic.
Connections:
- net WR_UART_RX: now reaches R6.2, U2.4 (A3)
- net IU_UART_TX: now reaches R4.2, U2.2 (A1)
- net IU_UART_RX: now reaches R5.2, U2.3 (A2)
- net WR_UART_TX: now reaches R7.2, U2.5 (A4)
Other:
- note added: "3.3V Output Switching Voltage Regulator:"
- note added: "CISPR 22 CLASS B EMI Filter:"
- note added: "Development:"
- note added: "Mounting Holes:"
- note added: "Operational Connectors:"
- note added: "Power Multiplexer:"
- note added: "System on a Chip (SoC):"
- note removed: "3.3V Output Switching Voltage Regulator"
- note removed: "CISPR 22 CLASS B EMI Filter"
- note removed: "Firmware Development, Debug and Recovery"
- note removed: "IU/USB Power Multiplexer"
- note removed: "Mounting Holes"
- note removed: "Operational Connectors"
- note removed: "System on a Chip (SoC)"
- moved on the sheet: C10, C11, C12, C13, C14, C15, C2, C3, C4, C5, C6, C7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

Commit message: Clean up KiCad schematic. Improve grounding in on PCB.
Parts:
- C2: value 1μF -> 0.1μF; symbol Project:Samsung_CL05A105KA5NQNC -> Project:Samsung_CL05B104KO5NNNC; LCSC Part # C52923 -> C1525; Part CL05A105KA5NQNC -> CL05B104KO5NNNC
- S1, S2: value SW_SPST -> SW_PUSH
Other:
- company: (none) -> Back in Thirty
- moved on the sheet: C2, C3, C4, C5, C6, R2, R3, R4, R5, R6, R7, U1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
